File: pcb/keyboard-x2-lumberjack-arm.kicad_pcb (KiCad board)
At the start: 2 copper layers, 285 x 94.2 mm, 144 parts, among them J1 16-pin USB-C Connector SMD, U1 STM32F103 Bluepill, or MiniF4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, U2 SN74LVC1T45DBV

Commit message: Update 20230326
Parts:
- added H5: ~, ProjectLocal:Bumpon_3M_F0502, F.Cu at (2.56, 2.56)
- added H6: ~, ProjectLocal:H_M2_Spacer_Hole, F.Cu at (2.15, 8.27)
- SW_1_1, SW_1_10, SW_1_11, SW_1_12, SW_1_2, SW_1_3, SW_1_4, SW_1_5, SW_1_6, SW_1_7, SW_1_8, SW_1_9, SW_2_1, SW_2_10, SW_2_11, SW_2_12, SW_2_2, SW_2_3, SW_2_4, SW_2_5, SW_2_6, SW_2_7, SW_2_8, SW_2_9, SW_3_1, SW_3_10, SW_3_11, SW_3_12, SW_3_2, SW_3_3, SW_3_4, SW_3_5, SW_3_6, SW_3_7, SW_3_8, SW_3_9, SW_4_1, SW_4_10, SW_4_11, SW_4_12, SW_4_2, SW_4_3, SW_4_4, SW_4_5, SW_4_6, SW_4_7, SW_4_8, SW_4_9, SW_5_1, SW_5_10, SW_5_11, SW_5_12, SW_5_2, SW_5_3, SW_5_4, SW_5_5, SW_5_6, SW_5_7, SW_5_8, SW_5_9: footprint ProjectLocal:SW_MX_PG1350_NoLed -> Library:CherryMX_Choc_Hotswap Single Side
Connections:
- D4 pad 2: Net-(D4-Pad2) -> unconnected-(D4-DOUT-Pad2)
- J1 pad A8: Net-(J1-PadA8) -> unconnected-(J1-SBU1-PadA8)
- J1 pad B8: Net-(J1-PadB8) -> unconnected-(J1-SBU2-PadB8)
- J1 pad S1: Net-(J1-PadS1) -> unconnected-(J1-SHIELD-PadS1)
- U1 pad 11: Net-(U1-Pad11) -> unconnected-(U1-B3-Pad11)
- U1 pad 12: Net-(U1-Pad12) -> unconnected-(U1-B4-Pad12)
- U1 pad 17: Net-(U1-Pad17) -> unconnected-(U1-B9-Pad17)
- U1 pad 21: Net-(U1-Pad21) -> unconnected-(U1-VBAT-Pad21)
- U1 pad 22: Net-(U1-Pad22) -> unconnected-(U1-C13-Pad22)
- U1 pad 23: Net-(U1-Pad23) -> unconnected-(U1-C14-Pad23)
- U1 pad 24: Net-(U1-Pad24) -> unconnected-(U1-C15-Pad24)
- U1 pad 25: Net-(U1-Pad25) -> unconnected-(U1-A0_or_RST-Pad25)
- U1 pad 26: Net-(U1-Pad26) -> unconnected-(U1-A1_or_A0-Pad26)
- U1 pad 27: Net-(U1-Pad27) -> unconnected-(U1-A2_or_A1-Pad27)
- U1 pad 28: Net-(U1-Pad28) -> unconnected-(U1-A3_or_A2-Pad28)
- U1 pad 36: Net-(U1-Pad36) -> unconnected-(U1-B11_or_B2-Pad36)
- U1 pad 37: Net-(U1-Pad37) -> unconnected-(U1-RST_or_B10-Pad37)
- U1 pad 6: Net-(U1-Pad6) -> unconnected-(U1-A9-Pad6)
Routing:
- net (no net): track 0.00 -> 1607.3 mm, vias 0 -> 4
- net Net-(D_5_1-A): track 132.8 -> 0.00 mm
- net Net-(D_5_12-A): track 121.1 -> 0.00 mm
- net Net-(D_5_2-A): track 119.4 -> 0.00 mm
- net Net-(D_1_1-A): track 118.0 -> 0.00 mm, vias 4 -> 0
- net Net-(D_5_11-A): track 107.3 -> 0.00 mm
- net Net-(D_5_3-A): track 101.3 -> 0.00 mm
- net Net-(D_4_2-A): track 97.6 -> 0.00 mm
- net Net-(D_5_10-A): track 89.6 -> 0.00 mm
- net Net-(D_5_4-A): track 87.0 -> 0.00 mm
- net Net-(D_1_3-A): track 76.1 -> 0.00 mm
- net Net-(D_3_3-A): track 75.5 -> 0.00 mm
- net Net-(D_5_9-A): track 75.2 -> 0.00 mm
- net Net-(D_5_5-A): track 69.2 -> 0.00 mm
- net Net-(D_2_4-A): track 59.6 -> 0.00 mm
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